Commit message: Add LiDAR sensor and Gazebo <-> ROS 2 /scan bridge

File: src/robot_description/urdf/robot.urdf.xacro (robot description, xacro)
@@ -1,25 +1,25 @@
 <?xml version="1.0"?>
 <robot name="robot_lab"
-       xmlns:xacro="http://www.ros.org/wiki/xacro">
+  xmlns:xacro="http://www.ros.org/wiki/xacro">
   <!-- ==================== BASE ==================== -->
   <link name="base_link">
     <visual>
-      <origin xyz="0 0 0.13"/>
-      <geometry>
-        <box size="0.40 0.30 0.10"/>
+      <origin xyz="0 0 0.13" />
+      <geometry>
+        <box size="0.40 0.30 0.10" />
       </geometry>
       <material name="blue">
-        <color rgba="0.1 0.3 0.8 1.0"/>
+        <color rgba="0.1 0.3 0.8 1.0" />
       </material>
     </visual>
     <collision>
-      <origin xyz="0 0 0.13"/>
-      <geometry>
-        <box size="0.40 0.30 0.10"/>
-      </geometry>
-    </collision>
-    <inertial>
-      <origin xyz="0 0 0.13"/>
-      <mass value="5.0"/>
+      <origin xyz="0 0 0.13" />
+      <geometry>
+        <box size="0.40 0.30 0.10" />
+      </geometry>
+    </collision>
+    <inertial>
+      <origin xyz="0 0 0.13" />
+      <mass value="5.0" />
       <inertia
         ixx="0.0417"
@@ -28,30 +28,30 @@
         iyy="0.0708"
         iyz="0"
-        izz="0.1042"/>
+        izz="0.1042" />
     </inertial>
   </link>
   <!-- ==================== LEFT WHEEL ==================== -->
   <joint name="left_wheel_joint" type="continuous">
-    <parent link="base_link"/>
-    <child link="left_wheel_link"/>
-    <origin xyz="0 0.17 0.08"/>
-    <axis xyz="0 1 0"/>
-    <dynamics damping="0.1"/>
+    <parent link="base_link" />
+    <child link="left_wheel_link" />
+    <origin xyz="0 0.17 0.08" />
+    <axis xyz="0 1 0" />
+    <dynamics damping="0.1" />
   </joint>
   <link name="left_wheel_link">
     <visual>
-      <origin rpy="1.5708 0 0"/>
-      <geometry>
-        <cylinder radius="0.08" length="0.04"/>
-      </geometry>
-    </visual>
-    <collision>
-      <origin rpy="1.5708 0 0"/>
-      <geometry>
-        <cylinder radius="0.08" length="0.04"/>
-      </geometry>
-    </collision>
-    <inertial>
-      <mass value="0.5"/>
+      <origin rpy="1.5708 0 0" />
+      <geometry>
+        <cylinder radius="0.08" length="0.04" />
+      </geometry>
+    </visual>
+    <collision>
+      <origin rpy="1.5708 0 0" />
+      <geometry>
+        <cylinder radius="0.08" length="0.04" />
+      </geometry>
+    </collision>
+    <inertial>
+      <mass value="0.5" />
       <inertia
         ixx="0.00087"
@@ -60,30 +60,30 @@
         iyy="0.00160"
         iyz="0"
-        izz="0.00087"/>
+        izz="0.00087" />
     </inertial>
   </link>
   <!-- ==================== RIGHT WHEEL ==================== -->
   <joint name="right_wheel_joint" type="continuous">
-    <parent link="base_link"/>
-    <child link="right_wheel_link"/>
-    <origin xyz="0 -0.17 0.08"/>
-    <axis xyz="0 1 0"/>
-    <dynamics damping="0.1"/>
+    <parent link="base_link" />
+    <child link="right_wheel_link" />
+    <origin xyz="0 -0.17 0.08" />
+    <axis xyz="0 1 0" />
+    <dynamics damping="0.1" />
   </joint>
   <link name="right_wheel_link">
     <visual>
-      <origin rpy="1.5708 0 0"/>
-      <geometry>
-        <cylinder radius="0.08" length="0.04"/>
-      </geometry>
-    </visual>
-    <collision>
-      <origin rpy="1.5708 0 0"/>
-      <geometry>
-        <cylinder radius="0.08" length="0.04"/>
-      </geometry>
-    </collision>
-    <inertial>
-      <mass value="0.5"/>
+      <origin rpy="1.5708 0 0" />
+      <geometry>
+        <cylinder radius="0.08" length="0.04" />
+      </geometry>
+    </visual>
+    <collision>
+      <origin rpy="1.5708 0 0" />
+      <geometry>
+        <cylinder radius="0.08" length="0.04" />
+      </geometry>
+    </collision>
+    <inertial>
+      <mass value="0.5" />
       <inertia
         ixx="0.00087"
@@ -92,26 +92,26 @@
         iyy="0.00160"
         iyz="0"
-        izz="0.00087"/>
+        izz="0.00087" />
     </inertial>
   </link>
   <!-- ==================== CASTER ==================== -->
   <joint name="caster_joint" type="fixed">
-    <parent link="base_link"/>
-    <child link="caster_link"/>
-    <origin xyz="-0.15 0 0.04"/>
+    <parent link="base_link" />
+    <child link="caster_link" />
+    <origin xyz="-0.15 0 0.04" />
   </joint>
   <link name="caster_link">
     <visual>
       <geometry>
-        <sphere radius="0.04"/>
-      </geometry>
-    </visual>
-    <collision>
-      <geometry>
-        <sphere radius="0.04"/>
-      </geometry>
-    </collision>
-    <inertial>
-      <mass value="0.1"/>
+        <sphere radius="0.04" />
+      </geometry>
+    </visual>
+    <collision>
+      <geometry>
+        <sphere radius="0.04" />
+      </geometry>
+    </collision>
+    <inertial>
+      <mass value="0.1" />
       <inertia
         ixx="0.000064"
@@ -120,7 +120,59 @@
         iyy="0.000064"
         iyz="0"
-        izz="0.000064"/>
-    </inertial>
-  </link>
+        izz="0.000064" />
+    </inertial>
+  </link>
+  <!-- ==================== LIDAR ==================== -->
+  <joint name="lidar_joint" type="fixed">
+    <parent link="base_link" />
+    <child link="lidar_link" />
+    <origin xyz="0 0 0.22" rpy="0 0 0" />
+  </joint>
+  <link name="lidar_link">
+    <visual>
+      <geometry>
+        <cylinder radius="0.035" length="0.03" />
+      </geometry>
+    </visual>
+    <collision>
+      <geometry>
+        <cylinder radius="0.035" length="0.03" />
+      </geometry>
+    </collision>
+    <inertial>
+      <mass value="0.1" />
+      <inertia
+        ixx="0.0001"
+        ixy="0"
+        ixz="0"
+        iyy="0.0001"
+        iyz="0"
+        izz="0.0001" />
+    </inertial>
+  </link>
+  <!-- ==================== GAZEBO LIDAR SENSOR ==================== -->
+  <gazebo reference="lidar_link">
+    <sensor name="lidar" type="gpu_lidar">
+      <topic>scan</topic>
+      <update_rate>10</update_rate>
+      <lidar>
+        <scan>
+          <horizontal>
+            <samples>360</samples>
+            <resolution>1</resolution>
+            <min_angle>-3.14159</min_angle>
+            <max_angle>3.14159</max_angle>
+          </horizontal>
+        </scan>
+        <range>
+          <min>0.12</min>
+          <max>8.0</max>
+          <resolution>0.01</resolution>
+        </range>
+      </lidar>
+      <always_on>true</always_on>
+      <visualize>true</visualize>
+    </sensor>
+  </gazebo>
   <!-- ==================== ROS 2 CONTROL ==================== -->
   <ros2_control name="GazeboSimSystem" type="system">
@@ -133,6 +185,6 @@
         <param name="max">20</param>
       </command_interface>
-      <state_interface name="position"/>
-      <state_interface name="velocity"/>
+      <state_interface name="position" />
+      <state_interface name="velocity" />
     </joint>
     <joint name="right_wheel_joint">
@@ -141,6 +193,6 @@
         <param name="max">20</param>
       </command_interface>
-      <state_interface name="position"/>
-      <state_interface name="velocity"/>
+      <state_interface name="position" />
+      <state_interface name="velocity" />
     </joint>
   </ros2_control>

Commit message: Move wheels forward to balance robot & change plane to gray

File: src/robot_description/urdf/robot.urdf.xacro (robot description, xacro)
@@ -35,5 +35,5 @@
     <parent link="base_link" />
     <child link="left_wheel_link" />
-    <origin xyz="0 0.17 0.08" />
+    <origin xyz="0.05 0.17 0.08" />
     <axis xyz="0 1 0" />
     <dynamics damping="0.1" />
@@ -67,5 +67,5 @@
     <parent link="base_link" />
     <child link="right_wheel_link" />
-    <origin xyz="0 -0.17 0.08" />
+    <origin xyz="0.05 -0.17 0.08" />
     <axis xyz="0 1 0" />
     <dynamics damping="0.1" />
